File: 02 Electronics/V0.2/3x3_board.kicad_pcb (KiCad board)
At the start: 2 copper layers, 69.1 x 104.8 mm, 124 parts, among them J1 Conn_01x04, J2 USB_B, J3 Conn_01x04, Q1 2N7002, Q10 BSS84, Q11 BSS84, Q12 BSS84, Q13 BSS84, Q2 2N7002, Q3 2N7002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

Commit message: add ctrlled to test all led routine + change some pins to pull up type
Other:
- net class Default removed
